Commit message: refactor kuka_kr6_r900 model: making all the accessories under kuka_kr6_r900 folder.

File: models/kuka_kr6_r900/urdf/kuka_kr6_r900_extrusion.urdf (robot description, URDF)
Before this commit: robot kr6_r900_mit_suction_gripper, 13 links, 12 joints
Links:
- removed link base_link
- removed link workspace_base_link
- link eef_base_link: geometry collision mesh filename=../meshes/asw_end_effector/collision/asw_hotend_end_effecto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 scale=.001 .001 .001; visual mesh filename=../meshes/asw_end_effector/visual/asw_hotend_end_effector.s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 scale=.001 .001 .001
- link robot_base_link: geometry collision mesh filename=../meshes/kr6_agilus/collision/base_link.stl; visual mesh filename=../meshes/kr6_agilus/visual/base_link.dae
- link robot_link_1: geometry collision mesh filename=../meshes/kr6_agilus/collision/link_1.stl; visual mesh filename=../meshes/kr6_agilus/visual/link_1.dae
- link robot_link_2: geometry collision mesh filename=../meshes/kr6r900sixx/collision/link_2.stl; visual mesh filename=../meshes/kr6r900sixx/visual/link_2.dae
- link robot_link_3: geometry collision mesh filename=../meshes/kr6_agilus/collision/link_3.stl; visual mesh filename=../meshes/kr6_agilus/visual/link_3.dae
- link robot_link_4: geometry collision mesh filename=../meshes/kr6r900sixx/collision/link_4.stl; visual mesh filename=../meshes/kr6r900sixx/visual/link_4.dae
- link robot_link_5: geometry collision mesh filename=../meshes/kr6_agilus/collision/link_5.stl; visual mesh filename=../meshes/kr6_agilus/visual/link_5.dae
- link robot_link_6: geometry collision mesh filename=../meshes/kr6_agilus/collision/link_6.stl; visual mesh filename=../meshes/kr6_agilus/visual/link_6.dae
Joints:
- removed joint world_to_base
- removed joint world_to_workspace
- joint eef_base_to_tcp: origin xyz=0.145336 0.001949 0.096286 rpy=0.0 1.57079632679 0.0 -> xyz=0.150539 0.001052 0.119157 rpy=0.0 1.57079632679 0.0
- joint robot_joint_a1: limit lower=-2.96705972839 upper=2.96705972839 effort=0 velocity=6.28318530718 -> lower=-1.57 upper=1.57 effort=0 velocity=6.28318530718
- joint robot_joint_a6: limit lower=-6.10865238198 upper=6.10865238198 effort=0 velocity=10.7337748998 -> lower=-3.14159 upper=3.14159 effort=0 velocity=10.7337748998

File: models/kuka_kr6_r900/urdf/kuka_kr6_r900_mit_suction_gripper.urdf (robot description, URDF)
Before this commit: robot kr6_r900_workspace, 16 links, 15 joints
Links:
- removed link material_feeder_material_feeder
- removed link material_feeder_mount_point
- removed link workspace_objects
- link eef_base_link: geometry collision mesh filename=../meshes/mit_arch_suction_gripper/collision/suction-grippe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 scale=.001 .001 .001; visual mesh filename=../meshes/mit_arch_suction_gripper/visual/suction-gripper_m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 scale=.001 .001 .001
- link robot_base_link: geometry collision mesh filename=../meshes/kr6_agilus/collision/base_link.stl; visual mesh filename=../meshes/kr6_agilus/visual/base_link.dae
- link robot_link_1: geometry collision mesh filename=../meshes/kr6_agilus/collision/link_1.stl; visual mesh filename=../meshes/kr6_agilus/visual/link_1.dae
- link robot_link_2: geometry collision mesh filename=../meshes/kr6r900sixx/collision/link_2.stl; visual mesh filename=../meshes/kr6r900sixx/visual/link_2.dae
- link robot_link_3: geometry collision mesh filename=../meshes/kr6_agilus/collision/link_3.stl; visual mesh filename=../meshes/kr6_agilus/visual/link_3.dae
- link robot_link_4: geometry collision mesh filename=../meshes/kr6r900sixx/collision/link_4.stl; visual mesh filename=../meshes/kr6r900sixx/visual/link_4.dae
- link robot_link_5: geometry collision mesh filename=../meshes/kr6_agilus/collision/link_5.stl; visual mesh filename=../meshes/kr6_agilus/visual/link_5.dae
- link robot_link_6: geometry collision mesh filename=../meshes/kr6_agilus/collision/link_6.stl; visual mesh filename=../meshes/kr6_agilus/visual/link_6.dae
Joints:
- removed joint link_3_to_link_3_mount_point
- removed joint mount_point_to_material_feeder
- removed joint workspace_baselink_to_objects
- joint eef_base_to_tcp: origin xyz=0.150539 0.001052 0.119157 rpy=0.0 1.57079632679 0.0 -> xyz=0.145336 0.001949 0.096286 rpy=0.0 1.57079632679 0.0
